File: fake-fan-simple/fake-fan-mk2.kicad_pcb (KiCad board)
At the start: 2 copper layers, 31 x 15 mm, 12 parts, among them J1 FIN1, J2 FOUT1, J3 SWD, U1 NJM12888, U2 STM32F030K6Tx

Commit message: 新版基板
Parts:
- added C6: 0.1u, Capacitor_SMD:C_0603_1608Metric, F.Cu at (23.8, 15.8)
- added G***: LOGO, ilks:LOGO, B.Cu at (32.5, 23.5)
- added R2: 22k, Resistor_SMD:R_0603_1608Metric, F.Cu at (17.4, 15.8)
- added R3: 22k, Resistor_SMD:R_0603_1608Metric, F.Cu at (20.6, 15.8)
- added R4: 22k, Resistor_SMD:R_0603_1608Metric, F.Cu at (38.0, 16.0)
- moved J3 0.40 mm to (21.0, 18.4)
Connections:
- J1 pad 3: /FAKE1 -> /FAKE_PULSE
- J1 pad 4: (no net) -> /PWMIN
- J2 pad 3: (no net) -> /FAN_PULSE
- J2 pad 4: /FAN1 -> /FAN_PWM
- U2 pad 12: (no net) -> /FAN_PWM
- U2 pad 13: (no net) -> /FAKE_PULSE
- U2 pad 21: /FAN1 -> /FAN_PULSE
- U2 pad 27: /FAKE1 -> (no net)
- U2 pad 7: (no net) -> /PWMIN_3V
Routing:
- net /PWMIN_3V: track 0.00 -> 24.1 mm, vias 0 -> 3
- net /FAN_PULSE: track 0.00 -> 23.6 mm, vias 0 -> 2
- net /FAKE_PULSE: track 0.00 -> 20.4 mm, vias 0 -> 1
- net /FAN1: track 13.8 -> 0.00 mm, vias 1 -> 0
- net /FAKE1: track 11.5 -> 0.00 mm
- net /FAN_PWM: track 0.00 -> 10.4 mm, vias 0 -> 1
- net /PWMIN: track 0.00 -> 2.64 mm
- net +3V3: track 42.2 -> 40.9 mm
- net +12V: track 35.7 -> 36.4 mm
- net GND: track 25.1 -> 25.3 mm, vias 5 -> 4
Other:
- board size 31 x 15 mm -> 31.5 x 15 mm
- board text added: "FakeFan4 @Hyper_beta"
- board text removed: "FakeFan3 @Hyper_beta"
