File: fake-fan-simple/fake-fan-mk2.sch (KiCad schematic (older format))
At the start: 12 parts, among them J1 FIN1, J2 FOUT1, J3 SWD, U1 NJM12888, U2 STM32F030K6Tx

Commit message: 新版基板
Parts:
- added C6: 0.1u, Capacitor_SMD:C_0603_1608Metric, symbol Device:C_Small
- added R2, R3, R?: 22k, Resistor_SMD:R_0603_1608Metric, symbol Device:R_Small
- gave numbers to parts that had none: 1
Connections:
- net labels added: FAKE_PULSE, FAN_PULSE, FAN_PWM, PWMIN, PWMIN_3V
- net labels removed: FAKE1, FAN1
- wire segments 72 -> 84
- no-connect marks 23 -> 19

Commit message: 回路更新
Parts:
- added TP1: TX, TestPoint:TestPoint_Pad_1.0x1.0mm, symbol Connector:TestPoint
- added TP2: RX, TestPoint:TestPoint_Pad_1.0x1.0mm, symbol Connector:TestPoint
- C1: value 0.47u -> 1u
- C5: value 0.1u -> 1u
- C6: value 0.1u -> 10u
- gave numbers to parts that had none: 1
Connections:
- net labels added: USART1_RX, USART1_TX
- wire segments 84 -> 88
- no-connect marks 19 -> 17
Changed lines of the file:
@@
 NoConn ~ 9250 3800
 NoConn ~ 9250 3700
-NoConn ~ 10350 3300
-NoConn ~ 10350 3400
 NoConn ~ 10350 3500
 NoConn ~ 10350 3600
@@
 NoConn ~ 10350 4000
 NoConn ~ 10350 4100
-NoConn ~ 10350 4300
+NoConn ~ 10350 4200
 NoConn ~ 9250 4000
 NoConn ~ 9250 4100
@@
 P 2350 1400
 F 0 "C1" H 2250 1350 50  0000 R CNN
-F 1 "0.47u" H 2250 1450 50  0000 R CNN
+F 1 "1u" H 2250 1450 50  0000 R CNN
 F 2 "Capacitor_SMD:C_0603_1608Metric" H 2350 1400 50  0001 C CNN
 F 3 "~" H 2350 1400 50  0001 C CNN
@@
 P 700 1400
 F 0 "C5" H 608 1354 50  0000 R CNN
-F 1 "0.1u" H 608 1445 50  0000 R CNN
+F 1 "1u" H 608 1445 50  0000 R CNN
 F 2 "Capacitor_SMD:C_0603_1608Metric" H 700 1400 50  0001 C CNN
 F 3 "~" H 700 1400 50  0001 C CNN
@@
 L Device:R_Small R2
 U 1 1 5F4F5E0C
-P 7850 3450
-F 0 "R2" V 7750 3450 50  0000 C CNN
-F 1 "22k" V 7950 3450 50  0000 C CNN
-F 2 "Resistor_SMD:R_0603_1608Metric" H 7850 3450 50  0001 C CNN
-F 3 "~" H 7850 3450 50  0001 C CNN
-	1    7850 3450
+P 5300 3800
+F 0 "R2" V 5200 3800 50  0000 C CNN
+F 1 "22k" V 5400 3800 50  0000 C CNN
+F 2 "Resistor_SMD:R_0603_1608Metric" H 5300 3800 50  0001 C CNN
+F 3 "~" H 5300 3800 50  0001 C CNN
+	1    5300 3800
 	1    0    0    1
 $EndComp
@@
 L Device:R_Small R3
 U 1 1 5F4F5E79
-P 7850 3950
-F 0 "R3" V 7750 3950 50  0000 C CNN
-F 1 "22k" V 7950 3950 50  0000 C CNN
-F 2 "Resistor_SMD:R_0603_1608Metric" H 7850 3950 50  0001 C CNN
-F 3 "~" H 7850 3950 50  0001 C CNN
-	1    7850 3950
+P 5300 4300
+F 0 "R3" V 5200 4300 50  0000 C CNN
+F 1 "22k" V 5400 4300 50  0000 C CNN
+F 2 "Resistor_SMD:R_0603_1608Metric" H 5300 4300 50  0001 C CNN
+F 3 "~" H 5300 4300 50  0001 C CNN
+	1    5300 4300
 	1    0    0    1
 $EndComp
@@
 L Device:C_Small C6
 U 1 1 5F4F5ED7
-P 8100 3950
-F 0 "C6" H 8008 3904 50  0000 R CNN
-F 1 "0.1u" H 8008 3995 50  0000 R CNN
-F 2 "Capacitor_SMD:C_0603_1608Metric" H 8100 3950 50  0001 C CNN
-F 3 "~" H 8100 3950 50  0001 C CNN
-	1    8100 3950
+P 5550 4300
+F 0 "C6" H 5458 4254 50  0000 R CNN
+F 1 "10u" H 5458 4345 50  0000 R CNN
+F 2 "Capacitor_SMD:C_0603_1608Metric" H 5550 4300 50  0001 C CNN
+F 3 "~" H 5550 4300 50  0001 C CNN
+	1    5550 4300
 	-1   0    0    1
 $EndComp
@@
 Wire Wire Line
 	4050 1250 4050 1150
-Text Label 7750 3200 2    50   ~ 0
+Text Label 5200 3550 2    50   ~ 0
 PWMIN
 $Comp
 L power:GND #PWR010
 U 1 1 5F504D42
-P 7850 4250
-F 0 "#PWR010" H 7850 4000 50  0001 C CNN
-F 1 "GND" V 7855 4122 50  0000 R CNN
-F 2 "" H 7850 4250 50  0001 C CNN
-F 3 "" H 7850 4250 50  0001 C CNN
-	1    7850 4250
-	1    0    0    -1
-$EndComp
-Wire Wire Line
-	7850 3350 7850 3200
-Wire Wire Line
-	7850 3200 7750 3200
-Wire Wire Line
-	7850 3550 7850 3750
-Wire Wire Line
-	7850 4050 7850 4150
-Wire Wire Line
-	7850 4150 8100 4150
-Wire Wire Line
-	8100 4150 8100 4050
-Connection ~ 7850 4150
-Wire Wire Line
-	7850 4150 7850 4250
-Wire Wire Line
-	8100 3850 8100 3750
-Wire Wire Line
-	8100 3750 7850 3750
-Connection ~ 7850 3750
-Wire Wire Line
-	7850 3750 7850 3850
+P 5300 4600
+F 0 "#PWR010" H 5300 4350 50  0001 C CNN
+F 1 "GND" V 5305 4472 50  0000 R CNN
+F 2 "" H 5300 4600 50  0001 C CNN
+F 3 "" H 5300 4600 50  0001 C CNN
+	1    5300 4600
+	1    0    0    -1
+$EndComp
+Wire Wire Line
+	5300 3700 5300 3550
+Wire Wire Line
+	5300 3550 5200 3550
+Wire Wire Line
+	5300 3900 5300 4100
+Wire Wire Line
+	5300 4400 5300 4500
+Wire Wire Line
+	5300 4500 5550 4500
+Wire Wire Line
+	5550 4500 5550 4400
+Connection ~ 5300 4500
+Wire Wire Line
+	5300 4500 5300 4600
+Wire Wire Line
+	5550 4200 5550 4100
+Wire Wire Line
+	5550 4100 5300 4100
+Connection ~ 5300 4100
+Wire Wire Line
+	5300 4100 5300 4200
 Text Label 10550 3200 0    50   ~ 0
 PWMIN_3V
-Text Label 8200 3750 0    50   ~ 0
+Text Label 5650 4100 0    50   ~ 0
 PWMIN_3V
 Wire Wire Line
-	8200 3750 8100 3750
-Connection ~ 8100 3750
+	5650 4100 5550 4100
+Connection ~ 5550 4100
 Wire Wire Line
 	10350 3200 10550 3200
@@
 Wire Wire Line
 	4750 1250 4850 1250
-Text Label 10550 4200 0    50   ~ 0
+Text Label 10550 4300 0    50   ~ 0
 FAN_PULSE
 Wire Wire Line
@@
 Text Label 10550 3800 0    50   ~ 0
 FAKE_PULSE
-Wire Wire Line
-	10350 4200 10550 4200
 NoConn ~ 9250 4300
-Text Label 8850 4600 3    50   ~ 0
+Text Label 4750 4450 3    50   ~ 0
 FAN_PULSE
 $Comp
-L Device:R_Small R?
+L Device:R_Small R4
 U 1 1 5F5329E4
-P 8850 4300
-F 0 "R?" V 8750 4300 50  0000 C CNN
-F 1 "22k" V 8950 4300 50  0000 C CNN
-F 2 "Resistor_SMD:R_0603_1608Metric" H 8850 4300 50  0001 C CNN
-F 3 "~" H 8850 4300 50  0001 C CNN
-	1    8850 4300
+P 4750 4150
+F 0 "R4" V 4650 4150 50  0000 C CNN
+F 1 "22k" V 4850 4150 50  0000 C CNN
+F 2 "Resistor_SMD:R_0603_1608Metric" H 4750 4150 50  0001 C CNN
+F 3 "~" H 4750 4150 50  0001 C CNN
+	1    4750 4150
 	1    0    0    1
 $EndComp
 $Comp
-L power:+3.3V #PWR?
+L power:+3.3V #PWR011
 U 1 1 5F532D13
-P 8850 4050
-F 0 "#PWR?" H 8850 3900 50  0001 C CNN
-F 1 "+3.3V" H 8865 4223 50  0000 C CNN
-F 2 "" H 8850 4050 50  0001 C CNN
-F 3 "" H 8850 4050 50  0001 C CNN
-	1    8850 4050
-	1    0    0    -1
-$EndComp
-Wire Wire Line
-	8850 4600 8850 4400
-Wire Wire Line
-	8850 4200 8850 4050
+P 4750 3900
+F 0 "#PWR011" H 4750 3750 50  0001 C CNN
+F 1 "+3.3V" H 4765 4073 50  0000 C CNN
+F 2 "" H 4750 3900 50  0001 C CNN
+F 3 "" H 4750 3900 50  0001 C CNN
+	1    4750 3900
+	1    0    0    -1
+$EndComp
+Wire Wire Line
+	4750 4450 4750 4250
+Wire Wire Line
+	4750 4050 4750 3900
+Wire Wire Line
+	10350 4300 10550 4300
+$Comp
+L Connector:TestPoint TP1
+U 1 1 5F509F32
+P 7700 3400
+F 0 "TP1" H 7758 3520 50  0000 L CNN
+F 1 "TX" H 7758 3429 50  0000 L CNN
+F 2 "TestPoint:TestPoint_Pad_1.0x1.0mm" H 7900 3400 50  0001 C CNN
+F 3 "~" H 7900 3400 50  0001 C CNN
+	1    7700 3400
+	1    0    0    -1
+$EndComp
+$Comp
+L Connector:TestPoint TP2
+U 1 1 5F50A050
+P 8000 3400
+F 0 "TP2" H 8058 3520 50  0000 L CNN
+F 1 "RX" H 8058 3429 50  0000 L CNN
+F 2 "TestPoint:TestPoint_Pad_1.0x1.0mm" H 8200 3400 50  0001 C CNN
+F 3 "~" H 8200 3400 50  0001 C CNN
+	1    8000 3400
+	1    0    0    -1
+$EndComp
+Text Label 8000 3500 3    50   ~ 0
+USART1_RX
+Text Label 7700 3500 3    50   ~ 0
+USART1_TX
+Wire Wire Line
+	7700 3500 7700 3400
+Wire Wire Line
+	8000 3400 8000 3500
+Text Label 10550 3400 0    50   ~ 0
+USART1_RX
+Text Label 10550 3300 0    50   ~ 0
+USART1_TX
+Wire Wire Line
+	10350 3300 10550 3300
+Wire Wire Line
+	10550 3400 10350 3400
 $EndSCHEMATC
